File: cz_8dt/cz_8dt.sch (KiCad schematic (older format))
At the start: 714 parts, among them IC1001 74LS09, IC1002 4001, IC1003 4049, IC101 MC4044, IC102 CD4053B, IC103 HD440072, IC104 4069, IC105 HA11720, IC106 74LS221, IC1101 74LS145, IC1102 74LS145, IC1103 74LS145, IC1104 7406, IC1105 74LS26, IC1106 7408, IC1201 7407, IC1202 7406, IC1203 74LS74, IC301 TA7348P, IC302 TA7348P, IC303 TA7347P, IC305 TA7348P, IC401 TA7348P, IC402 TA7348P, IC403 TA7347P, IC404 BA7001, IC404 TA7347P, IC601 X0065CE, IC602 74LS221, IC603 74LS221, IC604 74LS221, IC702 LM7805, IC801 TA7608CP, IC901 74159, IC902 74LS126, IC903 74LS126, IC904 74279, IC905 74279, IC906 74279, IC907 74LS126, IC908 74LS11, IC909 7406, Q1001 C1815, Q1002 C1815, Q101 C1815, Q103 C1815, Q104 C460, Q105 C1815, Q106 A454, Q107 C460, Q108 A454, Q109 C1815, Q1099 C1815, Q110 C1815, Q1101 A1015, Q1102 C1815, Q1103 C1815, Q1104 A1015, Q1105 C1815, Q1106 C1815, Q1107 A1015, Q1108 C1815, Q1109 C1815, Q111 A105, Q1110 C1815, Q1111 C1815, Q1112 A1015, Q1113 A1015, Q1114 A1015, Q1115 C1815, Q112 C1815, Q301 C1815, Q303 C1815, Q304 C1815, Q305 A1015, Q306 C1815, Q307 C1815, Q308 C1815, Q309 C1815, Q310 C1815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

Commit message: added front panel stuff
added front panel slider and led stuff
Parts:
- added D704: POWER_LED, symbol agg-kicad:LED
- added D901: TELOP_CUT, symbol agg-kicad:LED
- added D902: COMP, symbol agg-kicad:LED
- added D903: SUPER, symbol agg-kicad:LED
- added D904: VIDEO, symbol agg-kicad:LED
- added D905: VIN_1, symbol agg-kicad:LED
- added D906: VIN_2, symbol agg-kicad:LED
- added D907: VIN_3, symbol agg-kicad:LED
- added D908: MON_1, symbol agg-kicad:LED
- added D909: MON_2, symbol agg-kicad:LED
- added D910: MON_3, symbol agg-kicad:LED
- added D911: REC_OUT, symbol agg-kicad:LED
- added R182: 10R-18K, symbol Device:RTRIM
- added R342, R343, R344, R345, R346, R347, R704: R, symbol agg-kicad:R
- added R901, R902, R903, R904: 680R, symbol agg-kicad:R
- C?: value 2200uf? 35v ? -> 2200uf/35v
- R1164: value R_POT -> 470R
- R177: value R_POT -> 2.2K
Connections:
- wire segments 2724 -> 2834
- no-connect marks 47 -> 48
Other:
- note added: "5V comes\nthrough\nOrange wire"
- note added: "F2688CE PCB\n\n"
- note added: "F2689CE PCB\n\n"
- note added: "F2813CE PCB\n\n"
- note added: "G1 is 5V, but not \nconnected to anywhere"
- note added: "GND"
- note added: "Indicator LEDS\nAudio balance slider"
- note added: "Slider potentiomer for teloper area:\nCut\nout - in\n10R - 18K\n"
- note added: "from solder side"
- note added: "wire cut from the cable\nin main board side\n(would have been GND)"
- note removed: "Check D934 connections"
- note removed: "N1\n1\n2\nN2\n1\n2\n3\n4\n5\nN3\n1\n2\nN4\n1\n2\n3\n4\n5"
- note removed: "check this again?"
- note removed: "check\nfrom\nwhere ?"
- note removed: "check\nis H8 coming from this and\nalso from IC903-pin12?"
- note removed: "to Power\n LED"
- moved on the sheet: C902, D931, D932, D933, D934, D935, G_, IC907C, IC907D, R936

Commit message: added resistors/capacitors over the ICs
added resistors/capacitors that are over the ICs, so soldered to component side IC legs.
Parts:
- added C? (x32): 103, symbol agg-kicad:C
- added R? (x3): 150R, symbol agg-kicad:R
- added R? (x2): 560R, symbol agg-kicad:R
Connections:
- wire segments 2834 -> 2967
Other:
- note added: "Capacitor is\nover the IC"
- note added: "Capacitor is\nover the IC909"
- note added: "Capacitors are\nover the IC901"
- note added: "Capacitors are\nover the IC904"
- note added: "Capacitors are\nover the IC905"
- note added: "Capacitors are\nover the IC906"
- note added: "Capacitors/Resistors are\nover the IC1203"
- note added: "IC1203\npin 14\n\npin 7"
- note added: "IC902\npin 14\n\npin 7"
- note added: "IC903\npin 14\n\npin 7"
- note added: "IC904\npin 16\n\npin 8"
- note added: "IC905\npin 16\n\npin 8"
- note added: "IC906\npin 16\n\npin 8"
- note added: "IC907\npin 14\n\npin 7"
- note added: "IC908\npin 14\n\npin 7"
- note added: "IC909\npin 14\n\npin 7"
- note added: "pin 1"
- note added: "pin 2"
- note added: "pin 4"
- moved on the sheet: C628, IC901, R916, R917, R918, R919, R924

Commit message: added some missing stuff
Parts:
- removed C808: C, symbol agg-kicad:C
- added C101, C119: C, symbol agg-kicad:C
- added C102, C118, C808: CP, symbol agg-kicad:CP
- added unit 7 of IC1003
- added unit 7 of IC104
- added S901: TELOP, symbol agg-kicad:SWITCH_SPST
- added S902: COMP, symbol agg-kicad:SWITCH_SPST
- added S903: SUPER, symbol agg-kicad:SWITCH_SPST
- added S904: VIDEO, symbol agg-kicad:SWITCH_SPST
- added S905: VIN_1, symbol agg-kicad:SWITCH_SPST
- added S906: VIN_2, symbol agg-kicad:SWITCH_SPST
- added S907: VIN_3, symbol agg-kicad:SWITCH_SPST
- added S908: MON_1, symbol agg-kicad:SWITCH_SPST
- added S909: MON_2, symbol agg-kicad:SWITCH_SPST
- added S910: MON_3, symbol agg-kicad:SWITCH_SPST
- added S911: REC_OUT, symbol agg-kicad:SWITCH_SPST
Connections:
- net labels added: 9V, H1, O1, O2, O3, O4, O5, O6
- net labels removed: 12V?, ?V, IO1, IO2, IO3, O-_4, O-_5, O-_6
- wire segments 2967 -> 3021
Other:
- note added: "12V\n9V\n5V\nGND"
- note added: "All other IC 5V"
- note added: "Color Intensity"
- note added: "Color Tone"
- note added: "F2692CE PCB\n\n"
- note added: "G1 is 5V, \nbut not \nconnected \nto anywhere"
- note added: "H-position"
- note added: "H12 goes to GND\nin main PCB"
- note added: "IC102 9V\nIC104 9V\nIC105 9V"
- note added: "IC103 from 9V via resistor, -> 7.2V"
- note added: "IC601 from 12V via resistors\nIC801 12V\nIC1003 12V\n"
- note added: "Indicator LEDS, Push buttons and\nAudio balance slider"
- note added: "Near IC104"
- note added: "V-position"
- note added: "Video Adjust"
- note added: "backpanel\nadjustments (F2691CE)\n\n"
- note added: "drawn from solder side of pcb"
- note added: "near IC101"
- note removed: "12V\n7.2V\n5V\nGND"
- note removed: "G1 is 5V, but not \nconnected to anywhere"
- note removed: "Indicator LEDS\nAudio balance slider"
- note removed: "backpanel\nadjustments\n\n"
- note removed: "in trace side of pcb"
- moved on the sheet: C461, C806, D704, D901, D902, D903, D904, D905, D906, D907, D908, D909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

Commit message: double Q107 changed to Q102
Parts:
- Q102: renamed from Q107; value C460 -> C1815
Other:
- note removed: "Near IC104"
- note removed: "near IC101"
Changed lines of the file:
@@
 Connection ~ 15710 11980
 $Comp
-L Device:Q_NPN_BCE Q107
+L Device:Q_NPN_BCE Q102
 U 1 1 86BA2B8F
 P 10080 1320
-F 0 "Q107" V 9970 1440 50  0000 L CNN
-F 1 "C460" V 10060 1460 50  0000 L CNN
+F 0 "Q102" V 9970 1440 50  0000 L CNN
+F 1 "C1815" V 10060 1460 50  0000 L CNN
 F 2 "" H 10280 1420 50  0001 C CNN
 F 3 "~" H 10080 1320 50  0001 C CNN
@@
 Text Notes 16260 180  0    50   ~ 0
 H12 goes to GND\nin main PCB
-Text Notes 22610 6490 0    50   ~ 0
-Near IC104
-Text Notes 10420 1230 0    50   ~ 0
-near IC101
 $Comp
 L agg-kicad:CP C808

Commit message: rearranged into inside page. Added pdf version.
Other:
- note added: "G13 wire cut from the cable\nin main board side\n(would have been GND)"
- note added: "Not a typo!\nRCA input 3 and RGB21 audio\ninput channels are\nswapped connected,\nso this is clearly a design bug!"
- note added: "RGB21\nCSynch/\nCompVideo IN"
- note removed: "Not a typo!\nRCA input 3 and RGB21 audio input channels are\nswapped connected, so this is clearly a design bug!"
- note removed: "RGB21\nCSynch/CompVideo IN"
- note removed: "TP305"
- note removed: "wire cut from the cable\nin main board side\n(would have been GND)"
- moved on the sheet: A, B, C1005, C342, C343, C344, C345, C410, C427, C428, C461, C701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

Commit message: some comment texts updated in schematics
Other:
- note added: "EXT-S/COMPUTER: connects pins 1<->3 9<->11 5<->7 13 <->15\nVIDEO/COMPUTER: connects pins 2<->3, 10<->11, 6<->7, 14 <->15\nEXT-S/VIDEO: connects pins 3<->4, 11<->12, 7<->8, 15 <->16"
- note added: "RGB21\nR AUDIO IN"
- note added: "TV control Input and output\nSound-pin"
- note added: "audio balance slider\nfrom solder side"
- note removed: "EXT-S/COMPUTER - VIDEO/COMPUTER - EXT-S/VIDEO"
- note removed: "TV control Input and output"
- note removed: "from solder side"
Changed lines of the file:
@@
 Wire Notes Line
 	1390 21680 2360 21680
-Text Notes 1340 21110 0    50   ~ 0
+Text Notes 1370 20880 0    50   ~ 0
 switch to select audio mixing
-Text Notes 1020 21220 0    50   ~ 0
-EXT-S/COMPUTER - VIDEO/COMPUTER - EXT-S/VIDEO
+Text Notes 1110 21150 0    50   ~ 0
+EXT-S/COMPUTER: connects pins 1<->3 9<->11 5<->7 13 <->15\nVIDEO/COMPUTER: connects pins 2<->3, 10<->11, 6<->7, 14 <->15\nEXT-S/VIDEO: connects pins 3<->4,  11<->12, 7<->8, 15 <->16
 $Comp
 L agg-kicad:R R351
@@
 	2840 22170 2840 22240
 Text Notes 3370 22180 0    50   ~ 0
-TV control Input and output
+TV control Input and output\nSound-pin
 $Comp
 L power:GND #PWR0266
@@
 RGB21\nL AUDIO IN
 Text Notes 560  19200 0    50   ~ 0
-RGB21\nL AUDIO IN
+RGB21\nR AUDIO IN
 Text Notes 510  20700 0    50   ~ 0
 Not a typo!\nRCA input 3 and RGB21 audio\ninput channels are\nswapped connected,\nso this is clearly a design bug!
@@
 Text Notes 10800 1890 0    50   ~ 0
 GND
-Text Notes 11310 1770 0    50   ~ 0
-from solder side
+Text Notes 11250 1850 0    50   ~ 10
+audio balance slider\nfrom solder side
 Wire Notes Line
 	16910 16320 15410 16320
