File: CZ_VO_20PX_CPLD_VHD/X1_CZ_VO20PX_CPLD.sch (KiCad schematic (older format))
At the start: 112 parts, among them IC1 EMP7064_PLCC84, IC10 4538, IC100 ATmega328P-PU, IC101 ATmega328P-PU, IC102 4069, IC11 4013, IC120 LM1881, IC2 8251, IC3 74LS245, IC4 74LS393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

Commit message: Add files via upload
Parts:
- IC11: footprint Package_DIP:DIP-14_W10.16mm_LongPads -> Package_DIP:DIP-14_W7.62mm_Socket_LongPads
Changed lines of the file:
@@
 F 0 "IC11" H 19490 10581 50  0000 C CNN
 F 1 "4013" H 19490 10490 50  0000 C CNN
-F 2 "Package_DIP:DIP-14_W10.16mm_LongPads" H 19490 10100 50  0001 C CNN
+F 2 "Package_DIP:DIP-14_W7.62mm_Socket_LongPads" H 19490 10100 50  0001 C CNN
 F 3 "http://www.onsemi.com/pub/Collateral/MC14013B-D.PDF" H 19490 10100 50  0001 C CNN
 	1    19490 10100
@@
 F 0 "IC11" H 17130 15076 50  0000 L CNN
 F 1 "4013" H 17130 14985 50  0000 L CNN
-F 2 "Package_DIP:DIP-14_W10.16mm_LongPads" H 16900 15030 50  0001 C CNN
+F 2 "Package_DIP:DIP-14_W7.62mm_Socket_LongPads" H 16900 15030 50  0001 C CNN
 F 3 "http://www.onsemi.com/pub/Collateral/MC14013B-D.PDF" H 16900 15030 50  0001 C CNN
 	3    16900 15030

Commit message: corrected rx/tx mapping
corrected rx/tx mapping betwene atmega328p and 8251
Other:
- moved on the sheet: JP2, JP3
Changed lines of the file:
@@
 Wire Wire Line
 	9970 14070 9970 13970
+Text GLabel 13980 1840 3    50   Input ~ 0
+SW_RX
 Text GLabel 13690 2490 3    50   Input ~ 0
-SW_RX
-Text GLabel 13980 1840 3    50   Input ~ 0
 SW_TX
+Text GLabel 13980 1340 1    50   Input ~ 0
+RX
 Text GLabel 13690 1990 1    50   Input ~ 0
-RX
-Text GLabel 13980 1340 1    50   Input ~ 0
 TX
 $Comp
 L Jumper:Jumper_3_Open JP2
 U 1 1 6617A6BC
+P 13980 1590
+F 0 "JP2" V 13934 1677 50  0000 L CNN
+F 1 "Jumper_3_Open" V 14025 1677 50  0000 L CNN
+F 2 "Connector_PinHeader_2.54mm:PinHeader_1x03_P2.54mm_Vertical" H 13980 1590 50  0001 C CNN
+F 3 "~" H 13980 1590 50  0001 C CNN
+	1    13980 1590
+	0    1    1    0
+$EndComp
+$Comp
+L Jumper:Jumper_3_Open JP3
+U 1 1 6617A6BD
 P 13690 2240
-F 0 "JP2" V 13644 2327 50  0000 L CNN
+F 0 "JP3" V 13644 2327 50  0000 L CNN
 F 1 "Jumper_3_Open" V 13735 2327 50  0000 L CNN
 F 2 "Connector_PinHeader_2.54mm:PinHeader_1x03_P2.54mm_Vertical" H 13690 2240 50  0001 C CNN
@@
 	0    1    1    0
 $EndComp
-$Comp
-L Jumper:Jumper_3_Open JP3
-U 1 1 6617A6BD
-P 13980 1590
-F 0 "JP3" V 13934 1677 50  0000 L CNN
-F 1 "Jumper_3_Open" V 14025 1677 50  0000 L CNN
-F 2 "Connector_PinHeader_2.54mm:PinHeader_1x03_P2.54mm_Vertical" H 13980 1590 50  0001 C CNN
-F 3 "~" H 13980 1590 50  0001 C CNN
-	1    13980 1590
-	0    1    1    0
-$EndComp

Commit message: Add files via upload
Parts:
- removed C17: 100nF, Capacitor_THT:C_Disc_D5.0mm_W2.5mm_P5.00mm, symbol Device:C
- removed C203, C222: 100nF, Capacitor_THT:C_Disc_D4.3mm_W1.9mm_P5.00mm, symbol agg-kicad:C
- removed C23: 100nF, Capacitor_THT:C_Disc_D5.0mm_W2.5mm_P5.00mm, symbol agg-kicad:C
- removed IC11: 4013, Package_DIP:DIP-14_W7.62mm_Socket_LongPads, symbol 4xxx:4013
- removed IC120: LM1881, Package_DIP:DIP-8_W7.62mm, symbol Video:LM1881
- removed unit 2 of IC4
- removed IC7: 74LS02, Package_DIP:DIP-14_W7.62mm, symbol 74xx:74LS02
- removed JP8: Jumper_3_Open, Connector_PinHeader_2.54mm:PinHeader_1x03_P2.54mm_Vertical, symbol Jumper:Jumper_3_Open
- removed R230: 680K, Resistor_THT:R_Axial_DIN0207_L6.3mm_D2.5mm_P10.16mm_Horizontal, symbol agg-kicad:R
- removed SW3: CONN_02x08, Connector_PinHeader_2.54mm:PinHeader_2x08_P2.54mm_Vertical, symbol agg-kicad:CONN_02x08
- added unit 2 of IC102
- IC102: footprint (none) -> Package_DIP:DIP-14_W7.62mm
- Q2: value NPN (D637) or BC635 -> NPN (BC546); symbol Device:Q_NPN_BCE -> Device:Q_NPN_CBE
- R110: footprint Resistor_THT:R_Axial_DIN0207_L6.3mm_D2.5mm_P10.16mm_Horizontal -> Resistor_THT:R_Axial_DIN0207_L6.3mm_D2.5mm_P7.62mm_Horizontal
- R2, R5: footprint Resistor_THT:R_Axial_DIN0309_L9.0mm_D3.2mm_P12.70mm_Horizontal -> Resistor_THT:R_Axial_DIN0207_L6.3mm_D2.5mm_P7.62mm_Horizontal
- R400, R401, R403: footprint Resistor_THT:R_Axial_DIN0309_L9.0mm_D3.2mm_P12.70mm_Horizontal -> Resistor_THT:R_Axial_DIN0204_L3.6mm_D1.6mm_P7.62mm_Horizontal
Connections:
- net labels added: ~COMPOSITE_SYNCH, ~VHD9_PACKET_SYNC
- net labels removed: VHD9_INV, V_SYNCH
- wire segments 371 -> 320
- no-connect marks 19 -> 15
Other:
- moved on the sheet: IC102A, JP9
